File: CAD/Schematics/Updated Schematic 11-4-24/led20_updated_schematic_11_4_24.kicad_sch (KiCad schematic)
At the start: 31 parts

Commit message: Final revision of Updated Schematic 11-4-24
Parts:
- added TP13, TP14, TP15, TP16: ~, symbol Connector:TestPoint
- renumbered TP16 to TP17, TP14 to TP17, TP15 to TP18, TP17 to TP18, TP13 to TP19
Connections:
- net at U4.14 (LP_UART_RXD/GPIO4/LP_GPIO4/A4/MTMS): now also TP13.1
- net at U4.15 (LP_UART_TXD/LP_GPIO5/GPIO5/A5/MTDI): now also TP14.1
- net at U4.16 (LP_I2C_SDA/LP_GPIO6/GPIO6/A6/MTCK): now also TP15.1
- net at U4.17 (LP_I2C_SCL/LP_GPIO7/GPIO7/MTDO): now also TP16.1
Other:
- moved on the sheet: BZ1

Commit message: minor fixes
Parts:
- renumbered TP17 to TP19, TP18 to TP20, TP19 to TP21
Connections:
- net 3.3V Data (D3) is gone; now on net 3.3V Data (South): D2.3 (DIN)
- net 3.3V Data (D4) is gone; now on net 3.3V Data (North): D1.3 (DIN)
Changed lines of the file:
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@@
 		(title "LED20 Updated Schematic")
 		(date "2024-11-04")
-		(rev "2")
+		(rev "3")
 		(company "Team 01")
 		(comment 1 "Schematic of LED20 prototype")
@@
 	)
 	(rectangle
-		(start 184.15 21.59)
+		(start 181.61 21.59)
 		(end 229.87 96.52)
 		(stroke
@@
 	(text "LED Arrays"
 		(exclude_from_sim no)
-		(at 191.77 23.876 0)
+		(at 189.23 23.876 0)
 		(effects
 			(font
@@
 		)
 	)
-	(global_label "3.3V Data (D4)"
+	(global_label "3.3V Data (North)"
 		(shape input)
 		(at 203.2 44.45 180)
@@
 		)
 		(property "Intersheetrefs" "${INTERSHEET_REFS}"
-			(at 185.7006 44.45 0)
+			(at 183.0397 44.45 0)
 			(effects
 				(font
@@
 		)
 	)
-	(global_label "3.3V Data (D3)"
+	(global_label "3.3V Data (South)"
 		(shape input)
 		(at 203.2 80.01 180)
@@
 		)
 		(property "Intersheetrefs" "${INTERSHEET_REFS}"
-			(at 185.7006 80.01 0)
+			(at 182.7979 80.01 0)
 			(effects
 				(font
@@
 		(on_board yes)
 		(dnp no)
-		(property "Reference" "TP17"
+		(property "Reference" "TP19"
 			(at 113.538 48.26 90)
 			(effects
@@
 			(project "led20_updated_schematic_10_31_24"
 				(path "/967d5e27-871e-4805-83b6-90b8321a7dbd"
-					(reference "TP17")
+					(reference "TP19")
 					(unit 1)
 				)
@@
 		(on_board yes)
 		(dnp no)
-		(property "Reference" "TP18"
+		(property "Reference" "TP20"
 			(at 143.51 48.768 0)
 			(effects
@@
 			(project "led20_updated_schematic_10_31_24"
 				(path "/967d5e27-871e-4805-83b6-90b8321a7dbd"
-					(reference "TP18")
+					(reference "TP20")
 					(unit 1)
 				)
@@
 		(on_board yes)
 		(dnp no)
-		(property "Reference" "TP19"
+		(property "Reference" "TP21"
 			(at 142.24 103.378 0)
 			(effects
@@
 			(project "led20_updated_schematic_10_31_24"
 				(path "/967d5e27-871e-4805-83b6-90b8321a7dbd"
-					(reference "TP19")
+					(reference "TP21")
 					(unit 1)
 				)
