File: CAD/PCB/led20_updated_schematic_11_4_24.kicad_sch (KiCad schematic)
At the start: 32 parts, among them U3 Battery

Commit message: Updated PCB and Schematic
Changed schematic to include charging contact points and double checked pinouts on ICs
Parts:
- added U6: JST, Connector_JST:JST_PH_B2B-PH-K_1x02_P2.00mm_Vertical, symbol Connector:Conn_01x02_Socket
Connections:
- net GND: now also U4.16 (-), U6.2 (GND); no longer U4.15 (-)
- net VBATT: now also U4.15 (+); no longer U4.16 (+)
- net +5V IN: now reaches U4.14 (5V)
- net +5V IN: now also U6.1 (+5V_IN)
- no-connect marks 14 -> 13
Other:
- note added: "Charging Contact Points"
- moved on the sheet: C1, C2, C3, D1, TP17, TP18, TP19, TP20, U2

Commit message: Updated PCB and Schematic
Parts:
- BZ1: footprint (none) -> Buzzer_Beeper:Buzzer_12x9.5RM7.6
Changed lines of the file:
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@@
 	(title_block
 		(title "LED20 Updated Schematic")
-		(date "2024-11-04")
+		(date "2024-11-06")
 		(rev "2")
 		(company "Team 01")
@@
 			)
 		)
-		(property "Footprint" ""
+		(property "Footprint" "Buzzer_Beeper:Buzzer_12x9.5RM7.6"
 			(at 95.885 147.32 90)
 			(effects

Commit message: PCB and Schematic Update
Parts:
- removed BZ1: Piezo Buzzer, Buzzer_Beeper:Buzzer_12x9.5RM7.6, symbol Device:Buzzer
- removed U6: JST, Connector_JST:JST_PH_B2B-PH-K_1x02_P2.00mm_Vertical, symbol Connector:Conn_01x02_Socket
- added LS1: CMT-7525-80-SMT-TR, Led20:CMT-7525-80-SMT-TR_CUD, symbol 2024-11-12_02-31-52:CMT-7525-80-SMT-TR
- added U6, U7: B2B-PH-K-S, Connector_JST:JST_PH_B2B-PH-K_1x02_P2.00mm_Vertical, symbol 2024-11-12_01-25-46:B2B-PH-K-S
- D1: footprint LED_SMD:LED_SK6812MINI_PLCC4_3.5x3.5mm_P1.75mm -> Connector_JST:JST_PH_B3B-PH-K_1x03_P2.00mm_Vertical
- U3: footprint Connector_JST:JST_PH_B2B-PH-K_1x02_P2.00mm_Vertical -> (none)
Connections:
- net +5V: now also D1.1 (VDD); no longer D1.4 (VDD)
- net +5V IN: now also U6.1
- net 3.3V Data (D4): now also D1.2 (DIN); no longer D1.3 (DIN)
- net GND: now also D1.3 (VSS), LS1.2, U6.2, U7.2; no longer D1.2 (VSS), U3.2 (-)
- net VBATT: now also U7.1; no longer U3.1 (+)
- net at TP12.1, U4.1 (LP_GPIO0/GPIO0/A0/D0): now also LS1.1
Other:
- moved on the sheet: TP2

Commit message: PCB and Schematic Update
Updated PCB with traces and ground planes. Needs review. Battery symbol for schematic was removed - JST connector remains in its place.
Parts:
- removed U3: Battery, symbol Device:Battery
Other:
- note added: "BATT"
Changed lines of the file:
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@@
-	(wire
-		(pts
-			(xy 59.69 38.1) (xy 59.69 41.91)
-		)
-		(stroke
-			(width 0)
-			(type default)
-		)
-	)
 	(wire
 		(pts
@@
 	(wire
 		(pts
-			(xy 66.04 38.1) (xy 59.69 38.1)
-		)
-		(stroke
-			(width 0)
-			(type default)
-		)
-	)
-	(wire
-		(pts
 			(xy 74.93 111.76) (xy 80.01 111.76)
 		)
@@
 	(wire
 		(pts
-			(xy 59.69 48.26) (xy 59.69 44.45)
-		)
-		(stroke
-			(width 0)
-			(type default)
-		)
-	)
-	(wire
-		(pts
 			(xy 140.97 106.68) (xy 151.13 106.68)
 		)
@@
 		(pts
 			(xy 80.01 111.76) (xy 114.3 111.76)
-		)
-		(stroke
-			(width 0)
-			(type default)
-		)
-	)
-	(wire
-		(pts
-			(xy 66.04 48.26) (xy 59.69 48.26)
 		)
 		(stroke
@@
 		(exclude_from_sim no)
 		(at 52.07 26.162 0)
+		(effects
+			(font
+				(size 1.27 1.27)
+				(color 0 0 0 1)
+			)
+		)
+	)
+	(text "BATT"
+		(exclude_from_sim no)
+		(at 57.404 43.18 90)
 		(effects
 			(font
@@
 					(unit 1)
 				)
-			)
-		)
-	)
-	(symbol
-		(lib_id "Device:Battery")
-		(at 66.04 43.18 0)
-		(unit 1)
-		(exclude_from_sim no)
-		(in_bom yes)
-		(on_board yes)
-		(dnp no)
-		(property "Reference" "U3"
-			(at 63.5 33.528 0)
-			(effects
-				(font
-					(size 1.27 1.27)
-				)
-				(justify left)
-			)
-		)
-		(property "Value" "Battery"
-			(at 63.5 36.068 0)
-			(effects
-				(font
-					(size 1.27 1.27)
-				)
-				(justify left)
-			)
-		)
-		(property "Footprint" ""
-			(at 79.502 42.926 90)
-			(effects
-				(font
-					(size 1.27 1.27)
-				)
-				(hide yes)
-			)
-		)
-		(property "Datasheet" "~"
-			(at 66.04 41.656 90)
-			(effects
-				(font
-					(size 1.27 1.27)
-				)
-				(hide yes)
-			)
-		)
-		(property "Description" "Multiple-cell battery"
-			(at 66.04 43.18 0)
-			(effects
-				(font
-					(size 1.27 1.27)
-				)
-				(hide yes)
-			)
-		)
-		(pin "1"
-		)
-		(pin "2"
-		)
-		(instances
-			(project "led20_updated_schematic_11_4_24"
-				(path "/967d5e27-871e-4805-83b6-90b8321a7dbd"
-					(reference "U3")
-					(unit 1)
-				)

Commit message: PCB
Parts:
- renumbered TP23 to TP21
Other:
- note added: "Piezo Speaker"
- moved on the sheet: C1, C2, C3, C4, C5, D1, LS1, TP17, TP18, TP19, TP20, TP21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
