File: CAD/Schematics and PCB Layouts/LED20.kicad_pcb (KiCad board)
At the start: 2 copper layers, 30 x 35 mm, 32 parts, among them U6 B2B-PH-K-S, U7 B2B-PH-K-S

Commit message: Updated Directory and added new project contet
Parts:
- moved TP13 0.31 mm to (152.6, 65.9)
- moved TP14 0.12 mm to (151.2, 64.1)
Routing:
- net +5V: track 29.5 -> 27.1 mm
Changed lines of the file:
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@@
 		(rev "2")
 		(company "Team 01")
-		(comment 1 "PCB Layout of LED20 prototype")
+		(comment 1 "PCB Layout of LED20 ")
 	)
 	(layers
@@
 		(grid_origin 180.6375 59.95)
 		(pcbplotparams
-			(layerselection 0x0040000_7ffffffe)
-			(plot_on_all_layers_selection 0x7ffffff_80000001)
+			(layerselection 0x0001000_7ffffffe)
+			(plot_on_all_layers_selection 0x7fcffff_80000000)
 			(disableapertmacros no)
 			(usegerberextensions no)
@@
 			(subtractmaskfromsilk no)
 			(outputformat 4)
-			(mirror no)
+			(mirror yes)
 			(drillshape 0)
 			(scaleselection 1)
-			(outputdirectory "")
+			(outputdirectory "./")
 		)
 	)
@@
 		)
 		(fp_text user "${REFERENCE}"
-			(at 0 -2 90)
+			(at 0.008553 -1.763956 180)
 			(layer "F.Fab")
 			(effects
 				(font
-					(size 1 1)
-					(thickness 0.15)
+					(size 0.5 0.5)
+					(thickness 0.125)
 				)
 			)
@@
 		(tags "test point SMD pad")
 		(property "Reference" "TP16"
-			(at 0.007435 -1.428574 -0)
+			(at 0.007435 -1.428574 0)
 			(layer "B.SilkS")
 			(effects
@@
 	(footprint "TestPoint:TestPoint_Pad_D1.0mm"
 		(layer "F.Cu")
-		(at 152.333376 65.716062)
+		(at 152.5961 65.872827)
 		(descr "SMD pad as test Point, diameter 1.0mm")
 		(tags "test point SMD pad")
@@
 	(footprint "TestPoint:TestPoint_Pad_D1.0mm"
 		(layer "F.Cu")
-		(at 151.096977 64.084991)
+		(at 151.210712 64.128868)
 		(descr "SMD pad as test Point, diameter 1.0mm")
 		(tags "test point SMD pad")
@@
 		(tags "test point SMD pad")
 		(property "Reference" "TP6"
-			(at -0.294348 -2.913916 360)
+			(at -0.294348 -2.913916 0)
 			(layer "B.SilkS")
 			(effects
@@
 		)
 		(property "Value" "100n"
-			(at -3 0 360)
+			(at -3 0 0)
 			(layer "B.Fab")
 			(effects
@@
 	)
 	(gr_rect
-		(start 132.313079 63.386249)
-		(end 162.313079 98.386249)
+		(start 132.212322 63.338382)
+		(end 162.212322 98.338382)
 		(stroke
 			(width 0.05)
@@
 	)
 	(segment
-		(start 159.987862 74.416902)
-		(end 161.713079 74.416902)
+		(start 159.987862 88.960295)
+		(end 159.987862 74.416902)
 		(width 0.2)
 		(layer "F.Cu")
@@
 	)
 	(segment
-		(start 161.713079 74.416902)
-		(end 161.713079 87.235078)
-		(width 0.2)
-		(layer "F.Cu")
-		(net 5)
-	)
-	(segment
 		(start 158.812862 73.241902)
 		(end 159.987862 74.416902)
@@
 	)
 	(segment
-		(start 158.019656 92.996193)
-		(end 157.93581 92.912347)
+		(start 157.93581 91.012347)
+		(end 159.987862 88.960295)
 		(width 0.2)
 		(layer "F.Cu")
@@
 	)
 	(segment
-		(start 160.486961 94.960081)
-		(end 160.486961 93.087167)
+		(start 158.019656 92.996193)
+		(end 157.93581 92.912347)
 		(width 0.2)
 		(layer "F.Cu")
@@
 	)
 	(segment
-		(start 161.713079 87.235078)
-		(end 157.93581 91.012347)
+		(start 160.486961 94.960081)
+		(end 160.486961 93.087167)
 		(width 0.2)
 		(layer "F.Cu")
@@
 	)
 	(segment
-		(start 149.451438 65.716062)
-		(end 143.1775 71.99)
+		(start 152.5961 65.872827)
+		(end 149.294673 65.872827)
 		(width 0.2)
 		(layer "F.Cu")
@@
 	)
 	(segment
-		(start 152.333376 65.716062)
-		(end 149.451438 65.716062)
+		(start 149.294673 65.872827)
+		(end 143.1775 71.99)
 		(width 0.2)
 		(layer "F.Cu")
@@
 	)
 	(segment
-		(start 146.098531 63.988969)
+		(start 146.002509 64.084991)
 		(end 143.1775 66.91)
 		(width 0.2)
@@
 	(segment
 		(start 151.096977 64.084991)
-		(end 151.000955 63.988969)
-		(width 0.2)
-		(layer "F.Cu")
-		(net 15)
-	)
-	(segment
-		(start 151.000955 63.988969)
-		(end 146.098531 63.988969)
+		(end 146.002509 64.084991)
 		(width 0.2)
 		(layer "F.Cu")
