File: CAD/Schematics and PCB Layouts/LED20 v5.1/LED20.kicad_pcb (KiCad board)
At the start: 2 copper layers, 30 x 35 mm, 32 parts, among them U6 B2B-PH-K-S, U7 B2B-PH-K-S

Commit message: Update PCB
Updated test points, vias, and pcb traces. Added version number and team name to back of PCB.
Parts:
- moved TP15 0.14 mm to (133.6, 64.2)
- moved TP14 0.14 mm to (151.2, 64.3)
Other:
- board text added: "LED20 - V2 Team 01"
Changed lines of the file:
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@@
 	(footprint "TestPoint:TestPoint_Pad_D1.0mm"
 		(layer "F.Cu")
-		(at 133.570623 64.039269 180)
+		(at 133.558215 64.181695 180)
 		(descr "SMD pad as test Point, diameter 1.0mm")
 		(tags "test point SMD pad")
@@
 	(footprint "TestPoint:TestPoint_Pad_D1.0mm"
 		(layer "F.Cu")
-		(at 151.210712 64.128868)
+		(at 151.241689 64.264802)
 		(descr "SMD pad as test Point, diameter 1.0mm")
 		(tags "test point SMD pad")
@@
 		(layer "Edge.Cuts")
 	)
+	(gr_text "LED20 - V2\nTeam 01"
+		(at 161.273372 97.589096 0)
+		(layer "B.SilkS")
+		(effects
+			(font
+				(size 1 1)
+				(thickness 0.1)
+			)
+			(justify left bottom mirror)
+		)
+	)
 	(gr_text "LED\n"
 		(at 161.76029 74.012333 90)
@@
 	)
 	(segment
-		(start 139.608708 79.5332)
-		(end 141.1195 79.5332)
+		(start 158.828498 86.700433)
+		(end 158.828498 86.699486)
 		(width 0.2)
 		(layer "F.Cu")
@@
 	)
 	(segment
-		(start 158.828498 86.700433)
-		(end 158.828498 86.699486)
+		(start 137.921771 89.118373)
+		(end 137.921771 81.220137)
 		(width 0.2)
 		(layer "F.Cu")
@@
 	(segment
 		(start 143.656333 88.9547)
-		(end 143.656333 92.268932)
+		(end 142.422005 90.189028)
 		(width 0.2)
 		(layer "F.Cu")
@@
 	)
 	(segment
-		(start 137.921771 81.220137)
-		(end 139.608708 79.5332)
+		(start 142.422005 90.189028)
+		(end 142.422005 90.917602)
+		(width 0.2)
+		(layer "F.Cu")
+		(net 3)
+	)
+	(segment
+		(start 143.656333 88.9547)
+		(end 143.656333 92.268932)
 		(width 0.2)
 		(layer "F.Cu")
@@
 	)
 	(segment
-		(start 139.860182 90.189028)
-		(end 139.860182 91.056784)
+		(start 139.89668 91.093282)
+		(end 137.921771 89.118373)
 		(width 0.2)
 		(layer "F.Cu")
@@
 	)
 	(segment
-		(start 142.422005 90.917602)
-		(end 142.422005 90.189028)
-		(width 0.2)
-		(layer "F.Cu")
-		(net 3)
-	)
-	(segment
-		(start 141.1195 79.5332)
-		(end 142.6695 81.0832)
-		(width 0.2)
-		(layer "F.Cu")
-		(net 3)
-	)
-	(segment
-		(start 143.656333 88.9547)
-		(end 142.422005 90.189028)
-		(width 0.2)
-		(layer "F.Cu")
-		(net 3)
-	)
-	(segment
-		(start 139.860182 91.056784)
-		(end 139.89668 91.093282)
+		(start 143.656333 92.268932)
+		(end 145.542307 94.154906)
 		(width 0.2)
 		(layer "F.Cu")
@@
 	)
 	(segment
-		(start 143.656333 92.268932)
-		(end 145.542307 94.154906)
+		(start 137.921771 81.220137)
+		(end 139.608708 79.5332)
 		(width 0.2)
 		(layer "F.Cu")
@@
 	)
 	(segment
-		(start 137.921771 88.250617)
-		(end 137.921771 81.220137)
+		(start 141.1195 79.5332)
+		(end 142.6695 81.0832)
 		(width 0.2)
 		(layer "F.Cu")
@@
 	)
 	(segment
-		(start 139.860182 90.189028)
-		(end 137.921771 88.250617)
+		(start 139.608708 79.5332)
+		(end 141.1195 79.5332)
 		(width 0.2)
 		(layer "F.Cu")
@@
 	)
 	(segment
-		(start 146.002509 64.084991)
+		(start 145.822698 64.264802)
 		(end 143.1775 66.91)
 		(width 0.2)
@@
 	)
 	(segment
-		(start 151.096977 64.084991)
-		(end 146.002509 64.084991)
+		(start 151.241689 64.264802)
+		(end 145.822698 64.264802)
 		(width 0.2)
 		(layer "F.Cu")
@@
 	)
 	(segment
-		(start 133.570623 64.052054)
-		(end 133.570623 64.923123)
+		(start 133.570623 64.039269)
+		(end 133.570623 64.169287)
 		(width 0.2)
 		(layer "F.Cu")
@@
 	)
 	(segment
-		(start 133.570623 64.039269)
-		(end 133.570623 64.052054)
+		(start 133.558215 64.181695)
+		(end 133.558215 64.910715)
+		(width 0.2)
+		(layer "F.Cu")
+		(net 16)
+	)
+	(segment
+		(start 133.570623 64.169287)
+		(end 133.558215 64.181695)
 		(width 0.2)
 		(layer "F.Cu")
@@
 	)
 	(segment
-		(start 133.570623 64.923123)
+		(start 133.558215 64.910715)
 		(end 140.6375 71.99)
 		(width 0.2)
@@
 	)
 	(via
-		(at 133.570623 64.052054)
+		(at 133.558215 64.181695)
 		(size 0.6)
 		(drill 0.3)
