File: CAD/Schematics and PCB Layouts/LED20 V5.6/LED20.kicad_sch (KiCad schematic)
At the start: 24 parts, among them U3 MMBT4401LT1G, U6 B2B-PH-K-S, U7 B2B-PH-K-S

Commit message: Small revisions to final schematic, made pdf
Connections:
- no-connect marks 13 -> 15
Other:
- note added: "x20"
- note removed: "x10"
Changed lines of the file:
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@@
 	(title_block
 		(title "LED20 Final Schematic")
-		(date "2024-11-21")
-		(rev "5")
+		(date "2024-12-05")
+		(rev "5.6")
 		(company "Team 01")
 		(comment 1 "Schematic of LED20")
@@
 	)
 	(no_connect
+		(at 74.93 172.72)
+	)
+	(no_connect
 		(at 86.36 152.4)
+	)
+	(no_connect
+		(at 74.93 177.8)
 	)
 	(no_connect
@@
 		)
 	)
-	(text "x10"
+	(text "x20"
 		(exclude_from_sim no)
 		(at 222.758 38.354 0)
